File: Kicad/Arduino_EC.sch (KiCad schematic (older format))
At the start: 1 part

Commit message: Ready for 1st Review
Connections:
- net ECPump: now also ARD1.10 (SCL); no longer ARD1.5 (AnalogIn0)
Changed lines of the file:
@@
 Sheet 2 6
 Title ""
-Date "15 sep 2014"
+Date "16 sep 2014"
 Rev ""
 Comp ""
@@
 Wire Wire Line
 	5750 2800 6350 2800
-Text HLabel 2500 3550 0    60   Output ~ 0
+Text HLabel 2500 4550 0    60   Output ~ 0
 ECPump
 Text HLabel 6400 3600 2    60   Output ~ 0
@@
 	2500 2650 3550 2650
 Wire Wire Line
-	3550 3550 2500 3550
+	3550 4550 2500 4550
 $EndSCHEMATC

Commit message: Ready for Review
Parts:
- added TP9: CONN_1, symbol CONN_1
Connections:
- net GND_ARD: now also TP9.1
Changed lines of the file:
@@
 Sheet 2 6
 Title ""
-Date "16 sep 2014"
+Date "18 sep 2014"
 Rev ""
 Comp ""
@@
 Wire Wire Line
 	3550 4550 2500 4550
+$Comp
+L CONN_1 TP9
+U 1 1 5418B8C9
+P 3150 2900
+F 0 "TP9" H 3230 2900 40  0000 L CNN
+F 1 "CONN_1" H 3150 2955 30  0001 C CNN
+F 2 "" H 3150 2900 60  0000 C CNN
+F 3 "" H 3150 2900 60  0000 C CNN
+	1    3150 2900
+	1    0    0    -1
+$EndComp
+Wire Wire Line
+	3000 2650 3000 2900
+Connection ~ 3000 2650
 $EndSCHEMATC
