File: Kicad/Arduino_EC.sch (KiCad schematic (older format))
At the start: 1 part

Commit message: Started changes for Dev-Rev3
Parts:
- added D?: BLED, ~, symbol LED
- added R?: 499, ~, symbol R
Connections:
- net ECPump: now also ARD1.15 (Digital4); no longer ARD1.10 (SCL)
- net GND_ARD: now also R?.1
- net V+_ARD: now also D?.1 (A)
- net SDA: now reaches ARD1.9 (SDA)
- net MISO: no longer names the net of ARD1.23 (MISO)
- net MOSI: no longer names the net of ARD1.22 (MOSI)
- net SCLK: no longer names the net of ARD1.24 (SCK)
- net ~CS: no longer names the net of ARD1.18 (Digital7)
- net ~DR: no longer names the net of ARD1.17 (Digital6)
- net ~RESET: no longer names the net of ARD1.16 (Digital5)
- new net: D?.2 (K), R?.2
- new net SCL: ARD1.10 (SCL)
Other:
- note removed: "19,20,21 used by the Healthy pH Shield"
Changed lines of the file:
@@
 $Descr A4 11693 8268
 encoding utf-8
-Sheet 2 6
+Sheet 6 6
 Title ""
-Date "29 oct 2014"
+Date "14 nov 2014"
 Rev ""
 Comp ""
@@
 Comment4 ""
 $EndDescr
-Text HLabel 6350 2000 2    60   Output ~ 0
-SCLK
-Wire Wire Line
-	6350 2000 5750 2000
-Text HLabel 6350 2200 2    60   Input ~ 0
-MISO
-Text HLabel 6350 2400 2    60   Output ~ 0
-MOSI
-Text HLabel 6300 3200 2    60   Output ~ 0
-~CS
-Wire Wire Line
-	5750 2200 6350 2200
-Wire Wire Line
-	5750 2400 6350 2400
-Text HLabel 2500 4550 0    60   Output ~ 0
+Text HLabel 6800 3800 2    60   Output ~ 0
 ECPump
-Text HLabel 6400 3600 2    60   Output ~ 0
-~RESET
-Wire Wire Line
-	5750 3600 6400 3600
-Text HLabel 6450 3400 2    60   Input ~ 0
-~DR
-Wire Wire Line
-	5750 3400 6450 3400
 Text HLabel 2500 2450 0    60   Output ~ 0
 V+_ARD
@@
 	2500 2650 3550 2650
 Wire Wire Line
-	3550 4550 2500 4550
+	6800 3800 5750 3800
 Wire Wire Line
 	3550 2850 3200 2850
@@
 	3200 2850 3200 2650
 Connection ~ 3200 2650
+$Comp
+L LED D?
+U 1 1 5463AE5F
+P 2350 2000
+F 0 "D?" H 2350 2100 50  0000 C CNN
+F 1 "BLED" H 2350 1900 50  0000 C CNN
+F 2 "~" H 2350 2000 60  0000 C CNN
+F 3 "~" H 2350 2000 60  0000 C CNN
+	1    2350 2000
+	-1   0    0    1
+$EndComp
 Wire Wire Line
-	5750 3200 6300 3200
-Text Notes 5900 2750 0    60   ~ 0
-19,20,21 used by the Healthy pH Shield
+	2550 2000 2700 2000
+Wire Wire Line
+	2700 2000 2700 2450
+Connection ~ 2700 2450
+$Comp
+L R R?
+U 1 1 5463AE7B
+P 1600 2000
+F 0 "R?" V 1680 2000 40  0000 C CNN
+F 1 "499" V 1607 2001 40  0000 C CNN
+F 2 "~" V 1530 2000 30  0000 C CNN
+F 3 "~" H 1600 2000 30  0000 C CNN
+	1    1600 2000
+	0    -1   -1   0
+$EndComp
+Wire Wire Line
+	1850 2000 2150 2000
+Wire Wire Line
+	1350 2000 1100 2000
+Wire Wire Line
+	1100 2000 1100 2900
+Wire Wire Line
+	1100 2900 2650 2900
+Wire Wire Line
+	2650 2900 2650 2650
+Connection ~ 2650 2650
+Text HLabel 2900 4350 0    60   BiDi ~ 0
+SDA
+Wire Wire Line
+	2900 4350 3550 4350
+Text HLabel 2900 4550 0    60   BiDi ~ 0
+SCL
+Wire Wire Line
+	2900 4550 3550 4550
 $EndSCHEMATC
