File: Kicad/HealthypHShield.sch (KiCad schematic (older format))
At the start: 1 part

Commit message: Ready for 1st Review
Parts:
- added D?: LED, ~, symbol LED
- added R?: 1K, ~, symbol R
Connections:
- net AGND: now also R?.1
- net V+_WallWart: now also D?.1 (A)
- new net: D?.2 (K), R?.2
Changed lines of the file:
@@
 $Descr A4 11693 8268
 encoding utf-8
-Sheet 5 6
+Sheet 4 6
 Title ""
-Date "15 sep 2014"
+Date "16 sep 2014"
 Rev ""
 Comp ""
@@
 Wire Wire Line
 	4050 2800 4700 2800
+$Comp
+L LED D?
+U 1 1 5418A926
+P 4450 3200
+F 0 "D?" H 4450 3300 50  0000 C CNN
+F 1 "LED" H 4450 3100 50  0000 C CNN
+F 2 "~" H 4450 3200 60  0000 C CNN
+F 3 "~" H 4450 3200 60  0000 C CNN
+	1    4450 3200
+	0    1    1    0
+$EndComp
+$Comp
+L R R?
+U 1 1 5418A92C
+P 4450 3900
+F 0 "R?" V 4530 3900 40  0000 C CNN
+F 1 "1K" V 4457 3901 40  0000 C CNN
+F 2 "~" V 4380 3900 30  0000 C CNN
+F 3 "~" H 4450 3900 30  0000 C CNN
+	1    4450 3900
+	-1   0    0    1
+$EndComp
+Wire Wire Line
+	4450 3400 4450 3650
+Wire Wire Line
+	4450 4150 4450 4400
+$Comp
+L AGND #PWR?
+U 1 1 5418A935
+P 4450 4400
+F 0 "#PWR?" H 4450 4400 40  0001 C CNN
+F 1 "AGND" H 4450 4330 50  0000 C CNN
+F 2 "" H 4450 4400 60  0000 C CNN
+F 3 "" H 4450 4400 60  0000 C CNN
+	1    4450 4400
+	1    0    0    -1
+$EndComp
+Wire Wire Line
+	4450 3000 4450 2800
+Connection ~ 4450 2800
 $EndSCHEMATC

Commit message: Ready for Review
Parts:
- added TP13, TP14: CONN_1, symbol CONN_1
- gave numbers to parts that had none: 3
Connections:
- net AGND: now also TP13.1
- net V+_WallWart: now also TP14.1
Changed lines of the file:
@@
 Sheet 4 6
 Title ""
-Date "16 sep 2014"
+Date "18 sep 2014"
 Rev ""
 Comp ""
@@
 V+_WallWart
 $Comp
-L CONN_2 P?
+L CONN_2 P2
 U 1 1 53FA4108
 P 3950 2200
-F 0 "P?" V 3900 2200 40  0000 C CNN
+F 0 "P2" V 3900 2200 40  0000 C CNN
 F 1 "WallWartExtension" V 4100 2150 40  0000 C CNN
 F 2 "" H 3950 2200 60  0000 C CNN
@@
 $EndComp
 $Comp
-L AGND #PWR?
+L AGND #PWR02
 U 1 1 53FA4126
 P 3850 3150
-F 0 "#PWR?" H 3850 3150 40  0001 C CNN
+F 0 "#PWR02" H 3850 3150 40  0001 C CNN
 F 1 "AGND" H 3850 3080 50  0000 C CNN
 F 2 "" H 3850 3150 60  0000 C CNN
@@
 	4050 2800 4700 2800
 $Comp
-L LED D?
+L LED D2
 U 1 1 5418A926
 P 4450 3200
-F 0 "D?" H 4450 3300 50  0000 C CNN
+F 0 "D2" H 4450 3300 50  0000 C CNN
 F 1 "LED" H 4450 3100 50  0000 C CNN
 F 2 "~" H 4450 3200 60  0000 C CNN
@@
 $EndComp
 $Comp
-L R R?
+L R R9
 U 1 1 5418A92C
 P 4450 3900
-F 0 "R?" V 4530 3900 40  0000 C CNN
+F 0 "R9" V 4530 3900 40  0000 C CNN
 F 1 "1K" V 4457 3901 40  0000 C CNN
 F 2 "~" V 4380 3900 30  0000 C CNN
@@
 	4450 4150 4450 4400
 $Comp
-L AGND #PWR?
+L AGND #PWR03
 U 1 1 5418A935
 P 4450 4400
-F 0 "#PWR?" H 4450 4400 40  0001 C CNN
+F 0 "#PWR03" H 4450 4400 40  0001 C CNN
 F 1 "AGND" H 4450 4330 50  0000 C CNN
 F 2 "" H 4450 4400 60  0000 C CNN
@@
 	4450 3000 4450 2800
 Connection ~ 4450 2800
+$Comp
+L CONN_1 TP13
+U 1 1 5418BB40
+P 3600 2750
+F 0 "TP13" H 3680 2750 40  0000 L CNN
+F 1 "CONN_1" H 3600 2805 30  0001 C CNN
+F 2 "" H 3600 2750 60  0000 C CNN
+F 3 "" H 3600 2750 60  0000 C CNN
+	1    3600 2750
+	-1   0    0    1
+$EndComp
+$Comp
+L CONN_1 TP14
+U 1 1 54194E35
+P 4300 2650
+F 0 "TP14" H 4380 2650 40  0000 L CNN
+F 1 "CONN_1" H 4300 2705 30  0001 C CNN
+F 2 "" H 4300 2650 60  0000 C CNN
+F 3 "" H 4300 2650 60  0000 C CNN
+	1    4300 2650
+	1    0    0    -1
+$EndComp
+Wire Wire Line
+	4150 2650 4050 2650
+Connection ~ 4050 2650
+Wire Wire Line
+	3750 2750 3850 2750
+Connection ~ 3850 2750
 $EndSCHEMATC
