File: Kicad/HealthypHShield.sch (KiCad schematic (older format))
At the start: 3 parts, among them P2 WallWartExtension

Commit message: Started changes for Dev-Rev3
Parts:
- D2: value LED -> GLED
- R9: value 1K -> 499
Changed lines of the file:
@@
 $Descr A4 11693 8268
 encoding utf-8
-Sheet 4 6
+Sheet 3 6
 Title ""
-Date "29 oct 2014"
+Date "14 nov 2014"
 Rev ""
 Comp ""
@@
 P 4450 3200
 F 0 "D2" H 4450 3300 50  0000 C CNN
-F 1 "LED" H 4450 3100 50  0000 C CNN
+F 1 "GLED" H 4450 3100 50  0000 C CNN
 F 2 "~" H 4450 3200 60  0000 C CNN
 F 3 "~" H 4450 3200 60  0000 C CNN
@@
 P 4450 3900
 F 0 "R9" V 4530 3900 40  0000 C CNN
-F 1 "1K" V 4457 3901 40  0000 C CNN
+F 1 "499" V 4457 3901 40  0000 C CNN
 F 2 "~" V 4380 3900 30  0000 C CNN
 F 3 "~" H 4450 3900 30  0000 C CNN
