File: Kicad/Pumps_EC.sch (KiCad schematic (older format))
At the start: 4 parts, among them Q1 TIP122

Commit message: Ready for 1st Review
Parts:
- removed C14: 1u, ~, symbol C
- removed D1: 4004, ~, symbol DIODE
- removed Q1: TIP122, TO220, symbol TIP120
- removed R1: 2.2K, ~, symbol R
- added D?: 4004, ~, symbol DIODE
- added Q?: TIP122, TO220, symbol TIP120
- added R?: 2.2K, ~, symbol R
- added TP? (x3): CONN_1, symbol CONN_1
Connections:
- net ECPump: now also R?.1
- net GND: now also Q?.3 (E)
- net SW_ECPump: now also D?.1 (A), Q?.2 (C), TP?.1
- net V+_ARD: now also D?.2 (K), TP?.1
- new net: Q?.1 (B), R?.2, TP?.1
Changed lines of the file:
@@
 Sheet 3 6
 Title ""
-Date "15 sep 2014"
+Date "16 sep 2014"
 Rev ""
 Comp ""
@@
 Comment4 ""
 $EndDescr
+Text HLabel 7950 2650 2    60   Output ~ 0
+V+_ECPump
+Text HLabel 7950 3300 2    60   Input ~ 0
+SW_ECPump
 $Comp
-L TIP120 Q1
-U 1 1 53CBD30E
-P 3800 2650
-F 0 "Q1" H 3750 2500 40  0000 R CNN
-F 1 "TIP122" H 3800 2800 40  0000 R CNN
-F 2 "TO220" H 3680 2755 29  0001 C CNN
-F 3 "~" H 3800 2650 60  0000 C CNN
-	1    3800 2650
+L TIP120 Q?
+U 1 1 54188E8C
+P 5750 3600
+F 0 "Q?" H 5700 3450 40  0000 R CNN
+F 1 "TIP122" H 5750 3750 40  0000 R CNN
+F 2 "TO220" H 5630 3705 29  0001 C CNN
+F 3 "~" H 5750 3600 60  0000 C CNN
+	1    5750 3600
 	1    0    0    -1
 $EndComp
 $Comp
-L R R1
-U 1 1 53CBD483
-P 3100 2650
-F 0 "R1" V 3180 2650 40  0000 C CNN
-F 1 "2.2K" V 3107 2651 40  0000 C CNN
-F 2 "~" V 3030 2650 30  0000 C CNN
-F 3 "~" H 3100 2650 30  0000 C CNN
-	1    3100 2650
+L R R?
+U 1 1 54188E92
+P 5050 3600
+F 0 "R?" V 5130 3600 40  0000 C CNN
+F 1 "2.2K" V 5057 3601 40  0000 C CNN
+F 2 "~" V 4980 3600 30  0000 C CNN
+F 3 "~" H 5050 3600 30  0000 C CNN
+	1    5050 3600
 	0    -1   -1   0
 $EndComp
-Wire Wire Line
-	3350 2650 3600 2650
-Wire Wire Line
-	2000 2650 2850 2650
 $Comp
-L DIODE D1
-U 1 1 53CBD4B8
-P 4700 1500
-F 0 "D1" H 4700 1600 40  0000 C CNN
-F 1 "4004" H 4700 1400 40  0000 C CNN
-F 2 "~" H 4700 1500 60  0000 C CNN
-F 3 "~" H 4700 1500 60  0000 C CNN
-	1    4700 1500
-	0    1    1    0
+L DIODE D?
+U 1 1 54188E98
+P 7600 3000
+F 0 "D?" H 7600 3100 40  0000 C CNN
+F 1 "4004" H 7600 2900 40  0000 C CNN
+F 2 "~" H 7600 3000 60  0000 C CNN
+F 3 "~" H 7600 3000 60  0000 C CNN
+	1    7600 3000
+	0    -1   -1   0
 $EndComp
-Wire Wire Line
-	4700 1150 4700 1300
-Text HLabel 2000 2650 0    59   Input ~ 0
-ECPump
 $Comp
-L GND #PWR13
-U 1 1 53DC3138
-P 3900 3250
-F 0 "#PWR13" H 3900 3250 30  0001 C CNN
-F 1 "GND" H 3900 3180 30  0001 C CNN
-F 2 "" H 3900 3250 60  0000 C CNN
-F 3 "" H 3900 3250 60  0000 C CNN
-	1    3900 3250
+L GND #PWR?
+U 1 1 54188E9F
+P 5850 4200
+F 0 "#PWR?" H 5850 4200 30  0001 C CNN
+F 1 "GND" H 5850 4130 30  0001 C CNN
+F 2 "" H 5850 4200 60  0000 C CNN
+F 3 "" H 5850 4200 60  0000 C CNN
+	1    5850 4200
 	1    0    0    -1
 $EndComp
-Text HLabel 1750 1150 0    60   Input ~ 0
+Text HLabel 3700 2650 0    60   Input ~ 0
 V+_ARD
-Wire Wire Line
-	3900 2350 6000 2350
-Wire Wire Line
-	3900 2350 3900 2450
-Wire Wire Line
-	4700 1700 4700 2150
-Wire Wire Line
-	4700 2150 6000 2150
+Text HLabel 3650 4100 0    59   Output ~ 0
+GND_ARD
 $Comp
-L C C14
-U 1 1 53E26DDA
-P 2800 1500
-F 0 "C14" H 2800 1600 40  0000 L CNN
-F 1 "1u" H 2806 1415 40  0000 L CNN
-F 2 "~" H 2838 1350 30  0000 C CNN
-F 3 "~" H 2800 1500 60  0000 C CNN
-	1    2800 1500
-	-1   0    0    1
+L CONN_1 TP?
+U 1 1 54188EC4
+P 5700 2250
+F 0 "TP?" H 5780 2250 40  0000 L CNN
+F 1 "CONN_1" H 5700 2305 30  0001 C CNN
+F 2 "" H 5700 2250 60  0000 C CNN
+F 3 "" H 5700 2250 60  0000 C CNN
+	1    5700 2250
+	1    0    0    -1
 $EndComp
-Wire Wire Line
-	1750 1150 4700 1150
-Wire Wire Line
-	3900 2850 3900 3250
-Text HLabel 2000 3150 0    59   Output ~ 0
-GND_ARD
-Wire Wire Line
-	2000 3150 3900 3150
-Connection ~ 3900 3150
-Wire Wire Line
-	2800 1300 2800 1150
-Connection ~ 2800 1150
 $Comp
-L GND #PWR12
-U 1 1 53E3E3F6
-P 2800 1850
-F 0 "#PWR12" H 2800 1850 30  0001 C CNN
-F 1 "GND" H 2800 1780 30  0001 C CNN
-F 2 "" H 2800 1850 60  0000 C CNN
-F 3 "" H 2800 1850 60  0000 C CNN
-	1    2800 1850
+L CONN_1 TP?
+U 1 1 54188ECA
+P 6600 3050
+F 0 "TP?" H 6680 3050 40  0000 L CNN
+F 1 "CONN_1" H 6600 3105 30  0001 C CNN
+F 2 "" H 6600 3050 60  0000 C CNN
+F 3 "" H 6600 3050 60  0000 C CNN
+	1    6600 3050
+	1    0    0    -1
+$EndComp
+$Comp
+L CONN_1 TP?
+U 1 1 54188EDC
+P 5600 3050
+F 0 "TP?" H 5680 3050 40  0000 L CNN
+F 1 "CONN_1" H 5600 3105 30  0001 C CNN
+F 2 "" H 5600 3050 60  0000 C CNN
+F 3 "" H 5600 3050 60  0000 C CNN
+	1    5600 3050
 	1    0    0    -1
 $EndComp
 Wire Wire Line
-	2800 1700 2800 1850
-Text HLabel 6000 2150 2    60   Output ~ 0
-V+_ECPump
-Text HLabel 6000 2350 2    60   Input ~ 0
-SW_ECPump
+	5300 3600 5450 3600
+Wire Wire Line
+	5450 3600 5550 3600
+Wire Wire Line
+	3650 3600 4800 3600
+Wire Wire Line
+	5850 3300 6450 3300
+Wire Wire Line
+	6450 3300 7600 3300
+Wire Wire Line
+	7600 3300 7950 3300
+Wire Wire Line
+	5850 3300 5850 3400
+Wire Wire Line
+	3700 2650 5550 2650
+Wire Wire Line
+	5550 2650 7600 2650
+Wire Wire Line
+	7600 2650 7950 2650
+Wire Wire Line
+	5850 3800 5850 4100
+Wire Wire Line
+	5850 4100 5850 4200
+Wire Wire Line
+	3650 4100 5850 4100
+Connection ~ 5850 4100
+Wire Wire Line
+	7600 2800 7600 2650
+Connection ~ 7600 2650
+Wire Wire Line
+	7600 3200 7600 3300
+Connection ~ 7600 3300
+Wire Wire Line
+	5550 2250 5550 2650
+Connection ~ 5550 2650
+Wire Wire Line
+	6450 3050 6450 3300
+Connection ~ 6450 3300
+Wire Wire Line
+	5450 3050 5450 3600
+Connection ~ 5450 3600
+Text HLabel 3650 3600 0    59   Input ~ 0
+ECPump
 $EndSCHEMATC

Commit message: Ready for Review
Parts:
- removed TP?: CONN_1, symbol CONN_1
- gave numbers to parts that had none: 5
Changed lines of the file:
@@
 Sheet 3 6
 Title ""
-Date "16 sep 2014"
+Date "18 sep 2014"
 Rev ""
 Comp ""
@@
 SW_ECPump
 $Comp
-L TIP120 Q?
+L TIP120 Q1
 U 1 1 54188E8C
 P 5750 3600
-F 0 "Q?" H 5700 3450 40  0000 R CNN
+F 0 "Q1" H 5700 3450 40  0000 R CNN
 F 1 "TIP122" H 5750 3750 40  0000 R CNN
 F 2 "TO220" H 5630 3705 29  0001 C CNN
@@
 $EndComp
 $Comp
-L R R?
+L R R8
 U 1 1 54188E92
 P 5050 3600
-F 0 "R?" V 5130 3600 40  0000 C CNN
+F 0 "R8" V 5130 3600 40  0000 C CNN
 F 1 "2.2K" V 5057 3601 40  0000 C CNN
 F 2 "~" V 4980 3600 30  0000 C CNN
@@
 $EndComp
 $Comp
-L DIODE D?
+L DIODE D1
 U 1 1 54188E98
 P 7600 3000
-F 0 "D?" H 7600 3100 40  0000 C CNN
+F 0 "D1" H 7600 3100 40  0000 C CNN
 F 1 "4004" H 7600 2900 40  0000 C CNN
 F 2 "~" H 7600 3000 60  0000 C CNN
@@
 $EndComp
 $Comp
-L GND #PWR?
+L GND #PWR01
 U 1 1 54188E9F
 P 5850 4200
-F 0 "#PWR?" H 5850 4200 30  0001 C CNN
+F 0 "#PWR01" H 5850 4200 30  0001 C CNN
 F 1 "GND" H 5850 4130 30  0001 C CNN
 F 2 "" H 5850 4200 60  0000 C CNN
@@
 GND_ARD
 $Comp
-L CONN_1 TP?
+L CONN_1 TP11
 U 1 1 54188EC4
 P 5700 2250
-F 0 "TP?" H 5780 2250 40  0000 L CNN
+F 0 "TP11" H 5780 2250 40  0000 L CNN
 F 1 "CONN_1" H 5700 2305 30  0001 C CNN
 F 2 "" H 5700 2250 60  0000 C CNN
@@
 $EndComp
 $Comp
-L CONN_1 TP?
-U 1 1 54188ECA
-P 6600 3050
-F 0 "TP?" H 6680 3050 40  0000 L CNN
-F 1 "CONN_1" H 6600 3105 30  0001 C CNN
-F 2 "" H 6600 3050 60  0000 C CNN
-F 3 "" H 6600 3050 60  0000 C CNN
-	1    6600 3050
-	1    0    0    -1
-$EndComp
-$Comp
-L CONN_1 TP?
+L CONN_1 TP10
 U 1 1 54188EDC
 P 5600 3050
-F 0 "TP?" H 5680 3050 40  0000 L CNN
+F 0 "TP10" H 5680 3050 40  0000 L CNN
 F 1 "CONN_1" H 5600 3105 30  0001 C CNN
 F 2 "" H 5600 3050 60  0000 C CNN
@@
 $EndComp
 Wire Wire Line
-	5300 3600 5450 3600
-Wire Wire Line
-	5450 3600 5550 3600
+	5300 3600 5550 3600
 Wire Wire Line
 	3650 3600 4800 3600
 Wire Wire Line
-	5850 3300 6450 3300
-Wire Wire Line
-	6450 3300 7600 3300
-Wire Wire Line
-	7600 3300 7950 3300
+	5850 3300 7950 3300
 Wire Wire Line
 	5850 3300 5850 3400
 Wire Wire Line
-	3700 2650 5550 2650
+	3700 2650 7950 2650
 Wire Wire Line
-	5550 2650 7600 2650
-Wire Wire Line
-	7600 2650 7950 2650
-Wire Wire Line
-	5850 3800 5850 4100
-Wire Wire Line
-	5850 4100 5850 4200
+	5850 3800 5850 4200
 Wire Wire Line
 	3650 4100 5850 4100
@@
 Connection ~ 5550 2650
 Wire Wire Line
-	6450 3050 6450 3300
-Connection ~ 6450 3300
-Wire Wire Line
 	5450 3050 5450 3600
