File: Kicad/DigitalAccess_EC.sch (KiCad schematic (older format))
At the start: 11 parts, among them U2 MCP3901, X1 CRYSTAL

Commit message: Ready for layout review
Connections:
- net EC_GND renamed VGND
- net EC_Voltage renamed EC_Meas
Changed lines of the file:
@@
 	7200 1600 7200 1700
 Text HLabel 7900 3150 2    60   Input ~ 0
-EC_Voltage
+EC_Meas
 Text HLabel 7900 3250 2    60   Input ~ 0
-EC_GND
+VGND
 $EndSCHEMATC
