File: Kicad/DigitalAccess_EC.sch (KiCad schematic (older format))
At the start: 11 parts, among them U2 MCP3901, X1 CRYSTAL

Commit message: Started changes for Dev-Rev3
Parts:
- removed C1: 10u, ~, symbol C
- removed C2: .1u, ~, symbol C
- removed C4, C5: 18p, ~, symbol C
- removed C6: .1u, SM0805, symbol C
- removed C7: 1u, SM0805, symbol C
- removed C8: 10u, SM0805, symbol C
- removed L5: 1U, SM0805, symbol INDUCTOR
- removed R2: 1K, ~, symbol R
- removed U2: MCP3901, SSOP20, symbol MCP3901
- removed X1: CRYSTAL, ~, symbol CRYSTAL
- added .1u, C?: C, ~, symbol C
- added 3K (x2): R, ~, symbol R
- added R? (x4): 0, ~, symbol R
- added U?: MCP3221, ~, symbol MCP3221
- added U?: LB_MAX6003, symbol LB_MAX6003
Connections:
- net labels added: SCL, SDA
- net labels removed: AVdd, DVdd, MISO_ISO, MOSI_ISO, OSC1, OSC2, REFIN, SCLK_ISO, ~CS_ISO, ~DR, ~RESET
- wire segments 46 -> 25
