File: Kicad/HealthyEC.sch (KiCad schematic (older format))
At the start: 13 parts

Commit message: updated EC circuit
Parts:
- added R?: 499, ~, symbol R
- added TP?: TP, symbol CONN_1
Connections:
- net Arduino/~RESET: now also R?.1
- net EC/EC_Probe renamed EC/EC_V+
- net EC/EC_Probe_GND renamed EC/EC_Value
- new net DigitalAccess/~RESET: R?.2, TP?.1
Changed lines of the file:
@@
 Sheet 1 6
 Title ""
-Date "27 aug 2014"
+Date "15 sep 2014"
 Rev ""
 Comp ""
@@
 F0 "EC" 50
 F1 "EC.sch" 50
-F2 "EC_GND" O L 7350 2750 60
-F3 "EC_Probe" I R 9550 2350 60
-F4 "EC_Voltage" O L 7350 2550 60
-F5 "V+_WallWart" O L 7350 2150 60
-F6 "EC_Probe_GND" O R 9550 2550 60
+F2 "V+_WallWart" O L 7350 2150 60
+F3 "EC_V+" I R 9550 2350 60
+F4 "EC_Value" I R 9550 2550 60
+F5 "EC_V" I L 7350 2550 60
+F6 "EC_GND" I L 7350 2750 60
 $EndSheet
 $Sheet
@@
 	3550 4800 3400 4800
 Wire Wire Line
-	3400 4600 4400 4600
-Wire Wire Line
 	3400 5400 4400 5400
 Wire Wire Line
@@
 	3900 2150 7350 2150
 Connection ~ 5350 2150
+$Comp
+L R R?
+U 1 1 5415F8F0
+P 3800 4600
+F 0 "R?" V 3880 4600 40  0000 C CNN
+F 1 "499" V 3807 4601 40  0000 C CNN
+F 2 "~" V 3730 4600 30  0000 C CNN
+F 3 "~" H 3800 4600 30  0000 C CNN
+	1    3800 4600
+	0    -1   -1   0
+$EndComp
+Wire Wire Line
+	3550 4600 3400 4600
+Wire Wire Line
+	4050 4600 4400 4600
+$Comp
+L CONN_1 TP?
+U 1 1 5415F9F5
+P 4250 4500
+F 0 "TP?" H 4330 4500 40  0000 L CNN
+F 1 "TP" H 4250 4555 30  0001 C CNN
+F 2 "" H 4250 4500 60  0000 C CNN
+F 3 "" H 4250 4500 60  0000 C CNN
+	1    4250 4500
+	1    0    0    -1
+$EndComp
+Wire Wire Line
+	4100 4500 4100 4600
+Connection ~ 4100 4600
 $EndSCHEMATC

Commit message: Ready for 1st Review
Parts:
- removed TP?: TP, symbol CONN_1
Connections:
- net EC/EC_V+ renamed EC/EC_Probe+
- net EC/EC_Value renamed EC/EC_Probe-
Changed lines of the file:
@@
 Sheet 1 6
 Title ""
-Date "15 sep 2014"
+Date "16 sep 2014"
 Rev ""
 Comp ""
@@
 F0 "Pumps" 50
 F1 "Pumps_EC.sch" 50
-F2 "ECPump" I L 4400 5400 60
-F3 "V+_ARD" I L 4400 5550 60
-F4 "GND_ARD" O L 4400 5750 60
-F5 "V+_ECPump" O R 6500 5500 60
-F6 "SW_ECPump" I R 6500 5750 60
-$EndSheet
-$Sheet
-S 7350 2000 2200 1000
-U 53EF382C
-F0 "EC" 50
-F1 "EC.sch" 50
-F2 "V+_WallWart" O L 7350 2150 60
-F3 "EC_V+" I R 9550 2350 60
-F4 "EC_Value" I R 9550 2550 60
-F5 "EC_V" I L 7350 2550 60
-F6 "EC_GND" I L 7350 2750 60
+F2 "V+_ECPump" O R 6500 5500 60
+F3 "SW_ECPump" I R 6500 5750 60
+F4 "V+_ARD" I L 4400 5550 60
+F5 "GND_ARD" O L 4400 5750 60
+F6 "ECPump" I L 4400 5400 60
 $EndSheet
 $Sheet
@@
 $Comp
 L CONN_1 TP?
-U 1 1 53FA4584
-P 7200 2400
-F 0 "TP?" H 7280 2400 40  0000 L CNN
-F 1 "TP" H 7200 2455 30  0001 C CNN
-F 2 "" H 7200 2400 60  0000 C CNN
-F 3 "" H 7200 2400 60  0000 C CNN
-	1    7200 2400
-	1    0    0    -1
-$EndComp
-Wire Wire Line
-	7050 2400 7050 2550
-$Comp
-L CONN_1 TP?
 U 1 1 53FA45E3
 P 5500 2000
@@
 	4100 4500 4100 4600
 Connection ~ 4100 4600
+$Sheet
+S 7350 2000 2200 1000
+U 53EF382C
+F0 "EC" 50
+F1 "EC.sch" 50
+F2 "V+_WallWart" O L 7350 2150 60
+F3 "EC_V" I L 7350 2550 60
+F4 "EC_GND" I L 7350 2750 60
+F5 "EC_Probe+" I R 9550 2350 60
+F6 "EC_Probe-" I R 9550 2550 60
+$EndSheet
 $EndSCHEMATC

Commit message: Ready for Review
Parts:
- removed TP?: TP, symbol CONN_1
- gave numbers to parts that had none: 13
Connections:
- net EC/EC_Probe+: now also P1.4 (P4); no longer P1.1 (P1)
- net EC/EC_Probe-: now also P1.3 (P3); no longer P1.2 (P2)
- net Pumps/SW_ECPump: now also P1.1 (P1); no longer P1.4 (P4)
- net Pumps/V+_ECPump: now also P1.2 (P2); no longer P1.3 (P3)
Changed lines of the file:
@@
 Sheet 1 6
 Title ""
-Date "16 sep 2014"
+Date "18 sep 2014"
 Rev ""
 Comp ""
@@
 $EndSheet
 $Comp
-L CONN_4 P?
+L CONN_4 P1
 U 1 1 53F87484
 P 10750 4300
-F 0 "P?" V 10700 4300 50  0000 C CNN
+F 0 "P1" V 10700 4300 50  0000 C CNN
 F 1 "CONN_4" V 10800 4300 50  0000 C CNN
 F 2 "" H 10750 4300 60  0000 C CNN
 F 3 "" H 10750 4300 60  0000 C CNN
 	1    10750 4300
-	1    0    0    -1
+	1    0    0    1
 $EndComp
 $Sheet
@@
 $EndSheet
 $Comp
-L R R?
+L R R1
 U 1 1 53F9C5F1
 P 3800 3600
-F 0 "R?" V 3880 3600 40  0000 C CNN
+F 0 "R1" V 3880 3600 40  0000 C CNN
 F 1 "499" V 3807 3601 40  0000 C CNN
 F 2 "~" V 3730 3600 30  0000 C CNN
@@
 $EndComp
 $Comp
-L CONN_1 TP?
+L CONN_1 TP1
 U 1 1 53F9C600
 P 4200 3450
-F 0 "TP?" H 4280 3450 40  0000 L CNN
+F 0 "TP1" H 4280 3450 40  0000 L CNN
 F 1 "TP" H 4200 3505 30  0001 C CNN
 F 2 "" H 4200 3450 60  0000 C CNN
@@
 $EndComp
 $Comp
-L R R?
+L R R3
 U 1 1 53F9C710
 P 3800 3850
-F 0 "R?" V 3880 3850 40  0000 C CNN
+F 0 "R3" V 3880 3850 40  0000 C CNN
 F 1 "499" V 3807 3851 40  0000 C CNN
 F 2 "~" V 3730 3850 30  0000 C CNN
@@
 $EndComp
 $Comp
-L CONN_1 TP?
+L CONN_1 TP2
 U 1 1 53F9C716
 P 4200 3700
-F 0 "TP?" H 4280 3700 40  0000 L CNN
+F 0 "TP2" H 4280 3700 40  0000 L CNN
 F 1 "TP" H 4200 3755 30  0001 C CNN
 F 2 "" H 4200 3700 60  0000 C CNN
@@
 $EndComp
 $Comp
-L R R?
+L R R4
 U 1 1 53F9C770
 P 3800 4150
-F 0 "R?" V 3880 4150 40  0000 C CNN
+F 0 "R4" V 3880 4150 40  0000 C CNN
 F 1 "499" V 3807 4151 40  0000 C CNN
 F 2 "~" V 3730 4150 30  0000 C CNN
@@
 $EndComp
 $Comp
-L CONN_1 TP?
+L CONN_1 TP3
 U 1 1 53F9C776
 P 4200 4000
-F 0 "TP?" H 4280 4000 40  0000 L CNN
+F 0 "TP3" H 4280 4000 40  0000 L CNN
 F 1 "TP" H 4200 4055 30  0001 C CNN
 F 2 "" H 4200 4000 60  0000 C CNN
@@
 $EndComp
 $Comp
-L R R?
+L R R5
 U 1 1 53F9CA40
 P 3800 4400
-F 0 "R?" V 3880 4400 40  0000 C CNN
+F 0 "R5" V 3880 4400 40  0000 C CNN
 F 1 "499" V 3807 4401 40  0000 C CNN
 F 2 "~" V 3730 4400 30  0000 C CNN
@@
 $EndComp
 $Comp
-L CONN_1 TP?
+L CONN_1 TP4
 U 1 1 53F9CA46
 P 4200 4250
-F 0 "TP?" H 4280 4250 40  0000 L CNN
+F 0 "TP4" H 4280 4250 40  0000 L CNN
 F 1 "TP" H 4200 4305 30  0001 C CNN
 F 2 "" H 4200 4250 60  0000 C CNN
@@
 $EndComp
 $Comp
-L R R?
+L R R7
 U 1 1 53F9CAA0
 P 3800 4800
-F 0 "R?" V 3880 4800 40  0000 C CNN
+F 0 "R7" V 3880 4800 40  0000 C CNN
 F 1 "499" V 3807 4801 40  0000 C CNN
 F 2 "~" V 3730 4800 30  0000 C CNN
@@
 $EndComp
 $Comp
-L CONN_1 TP?
+L CONN_1 TP5
 U 1 1 53F9CAA6
 P 4200 4650
-F 0 "TP?" H 4280 4650 40  0000 L CNN
+F 0 "TP5" H 4280 4650 40  0000 L CNN
 F 1 "TP" H 4200 4705 30  0001 C CNN
 F 2 "" H 4200 4650 60  0000 C CNN
@@
 Wire Wire Line
 	10300 4150 10400 4150
-$Comp
-L CONN_1 TP?
-U 1 1 53FA45E3
-P 5500 2000
-F 0 "TP?" H 5580 2000 40  0000 L CNN
-F 1 "TP" H 5500 2055 30  0001 C CNN
-F 2 "" H 5500 2000 60  0000 C CNN
-F 3 "" H 5500 2000 60  0000 C CNN
-	1    5500 2000
-	1    0    0    -1
-$EndComp
-Wire Wire Line
-	5350 2000 5350 2150
 Wire Wire Line
 	3900 2150 7350 2150
-Connection ~ 5350 2150
-$Comp
-L R R?
+$Comp
+L R R6
 U 1 1 5415F8F0
 P 3800 4600
-F 0 "R?" V 3880 4600 40  0000 C CNN
+F 0 "R6" V 3880 4600 40  0000 C CNN
 F 1 "499" V 3807 4601 40  0000 C CNN
 F 2 "~" V 3730 4600 30  0000 C CNN
@@
 	4050 4600 4400 4600
 $Comp
-L CONN_1 TP?
+L CONN_1 TP6
 U 1 1 5415F9F5
 P 4250 4500
-F 0 "TP?" H 4330 4500 40  0000 L CNN
+F 0 "TP6" H 4330 4500 40  0000 L CNN
 F 1 "TP" H 4250 4555 30  0001 C CNN
 F 2 "" H 4250 4500 60  0000 C CNN

Commit message: Ready for layout review
Connections:
- net EC/EC_Probe- renamed DigitalAccess/VGND
Changed lines of the file:
@@
 F7 "V+_WallWart" O L 4400 2700 60
 F8 "~RESET" I L 4400 4600 60
-F9 "EC_Voltage" I R 6500 2550 60
-F10 "EC_GND" I R 6500 2750 60
+F9 "VGND" I R 6500 2750 60
+F10 "EC_Meas" I R 6500 2550 60
 $EndSheet
 $Comp
@@
 	1    0    0    -1
 $EndComp
-Wire Wire Line
-	3400 2700 4400 2700
-Wire Wire Line
-	3900 2150 3900 2700
-Connection ~ 3900 2700
-Wire Wire Line
-	7350 2750 6500 2750
-Wire Wire Line
-	7350 2550 6500 2550
-Wire Wire Line
-	3400 3600 3550 3600
-Wire Wire Line
-	4050 3600 4400 3600
-Wire Wire Line
-	3550 3850 3400 3850
-Wire Wire Line
-	4050 3850 4400 3850
-Wire Wire Line
-	4050 4150 4400 4150
-Wire Wire Line
-	4050 3450 4050 3600
-Wire Wire Line
-	4050 3700 4050 3850
-Wire Wire Line
-	4050 4000 4050 4150
-Wire Wire Line
-	4050 4250 4050 4400
-Wire Wire Line
-	4050 4400 4400 4400
-Wire Wire Line
-	3550 4400 3400 4400
-Wire Wire Line
-	3400 4150 3550 4150
-Wire Wire Line
-	4050 4650 4050 4800
-Wire Wire Line
-	4050 4800 4400 4800
-Wire Wire Line
-	3550 4800 3400 4800
-Wire Wire Line
-	3400 5400 4400 5400
-Wire Wire Line
-	3400 5550 4400 5550
-Wire Wire Line
-	3400 5750 4400 5750
-Wire Wire Line
-	6500 5750 10350 5750
-Wire Wire Line
-	10350 5750 10350 4450
-Wire Wire Line
-	10350 4450 10400 4450
-Wire Wire Line
-	6500 5500 10200 5500
-Wire Wire Line
-	10200 5500 10200 4350
-Wire Wire Line
-	10200 4350 10400 4350
-Wire Wire Line
-	10400 4250 10200 4250
-Wire Wire Line
-	10200 4250 10200 2550
-Wire Wire Line
-	10200 2550 9550 2550
-Wire Wire Line
-	9550 2350 10300 2350
-Wire Wire Line
-	10300 2350 10300 4150
-Wire Wire Line
-	10300 4150 10400 4150
-Wire Wire Line
-	3900 2150 7350 2150
 $Comp
 L R R6
@@
 	0    -1   -1   0
 $EndComp
-Wire Wire Line
-	3550 4600 3400 4600
-Wire Wire Line
-	4050 4600 4400 4600
 $Comp
 L CONN_1 TP6
@@
 	1    0    0    -1
 $EndComp
-Wire Wire Line
-	4100 4500 4100 4600
-Connection ~ 4100 4600
 $Sheet
 S 7350 2000 2200 1000
@@
 F1 "EC.sch" 50
 F2 "V+_WallWart" O L 7350 2150 60
-F3 "EC_V" I L 7350 2550 60
-F4 "EC_GND" I L 7350 2750 60
-F5 "EC_Probe+" I R 9550 2350 60
-F6 "EC_Probe-" I R 9550 2550 60
+F3 "EC_Probe+" I R 9550 2350 60
+F4 "VGND" I L 7350 2750 60
+F5 "EC_Meas" O L 7350 2550 60
 $EndSheet
+Wire Wire Line
+	3400 2700 4400 2700
+Wire Wire Line
+	3900 2150 3900 2700
+Connection ~ 3900 2700
+Wire Wire Line
+	7350 2750 6500 2750
+Wire Wire Line
+	7350 2550 6500 2550
+Wire Wire Line
+	3400 3600 3550 3600
+Wire Wire Line
+	4050 3600 4400 3600
+Wire Wire Line
+	3550 3850 3400 3850
+Wire Wire Line
+	4050 3850 4400 3850
+Wire Wire Line
+	4050 4150 4400 4150
+Wire Wire Line
+	4050 3450 4050 3600
+Wire Wire Line
+	4050 3700 4050 3850
+Wire Wire Line
+	4050 4000 4050 4150
+Wire Wire Line
+	4050 4250 4050 4400
+Wire Wire Line
+	4050 4400 4400 4400
+Wire Wire Line
+	3550 4400 3400 4400
+Wire Wire Line
+	3400 4150 3550 4150
+Wire Wire Line
+	4050 4650 4050 4800
+Wire Wire Line
+	4050 4800 4400 4800
+Wire Wire Line
+	3550 4800 3400 4800
+Wire Wire Line
+	3400 5400 4400 5400
+Wire Wire Line
+	3400 5550 4400 5550
+Wire Wire Line
+	3400 5750 4400 5750
+Wire Wire Line
+	6500 5750 10350 5750
+Wire Wire Line
+	10350 5750 10350 4450
+Wire Wire Line
+	10350 4450 10400 4450
+Wire Wire Line
+	6500 5500 10200 5500
+Wire Wire Line
+	10200 5500 10200 4350
+Wire Wire Line
+	10200 4350 10400 4350
+Wire Wire Line
+	10400 4250 10200 4250
+Wire Wire Line
+	9550 2350 10300 2350
+Wire Wire Line
+	10300 2350 10300 4150
+Wire Wire Line
+	10300 4150 10400 4150
+Wire Wire Line
+	3900 2150 7350 2150
+Wire Wire Line
+	3550 4600 3400 4600
+Wire Wire Line
+	4050 4600 4400 4600
+Wire Wire Line
+	4100 4500 4100 4600
+Connection ~ 4100 4600
+Wire Wire Line
+	7100 2750 7100 3300
+Wire Wire Line
+	7100 3300 10200 3300
+Connection ~ 7100 2750
+Wire Wire Line
+	10200 3300 10200 4250
 $EndSCHEMATC
