File: Kicad/HealthyEC.sch (KiCad schematic (older format))
At the start: 7 parts, among them P1 CONN_4

Commit message: Started changes for Dev-Rev3
Parts:
- removed R1, R3, R4, R5, R6, R7: 499, ~, symbol R
Changed lines of the file:
@@
 Sheet 1 6
 Title ""
-Date "29 oct 2014"
+Date "14 nov 2014"
 Rev ""
 Comp ""
@@
 Comment4 ""
 $EndDescr
-$Sheet
-S 950  3250 2450 3400
-U 53EF3667
-F0 "Arduino" 50
-F1 "Arduino_EC.sch" 50
-F2 "SCLK" O R 3400 3600 60
-F3 "MISO" I R 3400 3850 60
-F4 "MOSI" O R 3400 4150 60
-F5 "~CS" O R 3400 4400 60
-F6 "ECPump" O R 3400 5400 60
-F7 "~RESET" O R 3400 4600 60
-F8 "~DR" I R 3400 4800 60
-F9 "V+_ARD" O R 3400 5550 60
-F10 "GND_ARD" I R 3400 5750 60
-$EndSheet
 $Sheet
 S 4400 5200 2100 800
@@
 $EndComp
 $Sheet
-S 4400 2400 2100 2500
-U 53EF37AC
-F0 "DigitalAccess" 50
-F1 "DigitalAccess_EC.sch" 50
-F2 "MOSI_ISO" I L 4400 4150 60
-F3 "MISO_ISO" O L 4400 3850 60
-F4 "SCLK_ISO" I L 4400 3600 60
-F5 "~CS_ISO" I L 4400 4400 60
-F6 "~DR" O L 4400 4800 60
-F7 "V+_WallWart" O L 4400 2700 60
-F8 "~RESET" I L 4400 4600 60
-F9 "VGND" I R 6500 2750 60
-F10 "EC_Meas" I R 6500 2550 60
-$EndSheet
-$Comp
-L R R1
-U 1 1 53F9C5F1
-P 3800 3600
-F 0 "R1" V 3880 3600 40  0000 C CNN
-F 1 "499" V 3807 3601 40  0000 C CNN
-F 2 "~" V 3730 3600 30  0000 C CNN
-F 3 "~" H 3800 3600 30  0000 C CNN
-	1    3800 3600
-	0    -1   -1   0
-$EndComp
-$Comp
-L R R3
-U 1 1 53F9C710
-P 3800 3850
-F 0 "R3" V 3880 3850 40  0000 C CNN
-F 1 "499" V 3807 3851 40  0000 C CNN
-F 2 "~" V 3730 3850 30  0000 C CNN
-F 3 "~" H 3800 3850 30  0000 C CNN
-	1    3800 3850
-	0    -1   -1   0
-$EndComp
-$Comp
-L R R4
-U 1 1 53F9C770
-P 3800 4150
-F 0 "R4" V 3880 4150 40  0000 C CNN
-F 1 "499" V 3807 4151 40  0000 C CNN
-F 2 "~" V 3730 4150 30  0000 C CNN
-F 3 "~" H 3800 4150 30  0000 C CNN
-	1    3800 4150
-	0    -1   -1   0
-$EndComp
-$Comp
-L R R5
-U 1 1 53F9CA40
-P 3800 4400
-F 0 "R5" V 3880 4400 40  0000 C CNN
-F 1 "499" V 3807 4401 40  0000 C CNN
-F 2 "~" V 3730 4400 30  0000 C CNN
-F 3 "~" H 3800 4400 30  0000 C CNN
-	1    3800 4400
-	0    -1   -1   0
-$EndComp
-$Comp
-L R R7
-U 1 1 53F9CAA0
-P 3800 4800
-F 0 "R7" V 3880 4800 40  0000 C CNN
-F 1 "499" V 3807 4801 40  0000 C CNN
-F 2 "~" V 3730 4800 30  0000 C CNN
-F 3 "~" H 3800 4800 30  0000 C CNN
-	1    3800 4800
-	0    -1   -1   0
-$EndComp
-$Comp
-L R R6
-U 1 1 5415F8F0
-P 3800 4600
-F 0 "R6" V 3880 4600 40  0000 C CNN
-F 1 "499" V 3807 4601 40  0000 C CNN
-F 2 "~" V 3730 4600 30  0000 C CNN
-F 3 "~" H 3800 4600 30  0000 C CNN
-	1    3800 4600
-	0    -1   -1   0
-$EndComp
-$Sheet
 S 7350 2000 2200 1000
 U 53EF382C
@@
 F2 "V+_WallWart" O L 7350 2150 60
 F3 "EC_Probe+" I R 9550 2350 60
-F4 "VGND" I L 7350 2750 60
-F5 "EC_Meas" O L 7350 2550 60
+F4 "EC_Meas" O L 7350 2550 60
+F5 "VGND" I L 7350 2750 60
 $EndSheet
 Wire Wire Line
@@
 Wire Wire Line
 	7350 2550 6500 2550
-Wire Wire Line
-	3400 3600 3550 3600
-Wire Wire Line
-	4050 3600 4400 3600
-Wire Wire Line
-	3550 3850 3400 3850
-Wire Wire Line
-	4050 3850 4400 3850
-Wire Wire Line
-	4050 4150 4400 4150
-Wire Wire Line
-	4050 4400 4400 4400
-Wire Wire Line
-	3550 4400 3400 4400
-Wire Wire Line
-	3400 4150 3550 4150
-Wire Wire Line
-	4050 4800 4400 4800
-Wire Wire Line
-	3550 4800 3400 4800
 Wire Wire Line
 	3400 5400 4400 5400
@@
 	3900 2150 7350 2150
 Wire Wire Line
-	3550 4600 3400 4600
-Wire Wire Line
-	4050 4600 4400 4600
-Connection ~ 4100 4600
-Wire Wire Line
 	7100 2750 7100 3300
 Wire Wire Line
@@
 Wire Wire Line
 	10200 3300 10200 4250
+$Sheet
+S 4400 2400 2100 2500
+U 53EF37AC
+F0 "DigitalAccess" 50
+F1 "DigitalAccess_EC.sch" 50
+F2 "V+_WallWart" I L 4400 2700 60
+F3 "VGND" I R 6500 2750 60
+F4 "SCL" B L 4400 3700 60
+F5 "SDA" B L 4400 3950 60
+F6 "EC_Meas" I R 6500 2550 60
+$EndSheet
+$Sheet
+S 950  3250 2450 3400
+U 53EF3667
+F0 "Arduino" 50
+F1 "Arduino_EC.sch" 50
+F2 "ECPump" O R 3400 5400 60
+F3 "V+_ARD" O R 3400 5550 60
+F4 "GND_ARD" I R 3400 5750 60
+$EndSheet
 $EndSCHEMATC
