File: Kicad/HealthyEC.kicad_pcb (KiCad board)
At the start: 2 copper layers, 68.6 x 53.3 mm, 59 parts, among them P1 CONN_4, P2 WallWartExtension, Q1 TIP122, U1 MCP6244, U2 MCP3901, X1 CRYSTAL

Commit message: Ready for layout review
Parts:
- Q1: footprint TO220 -> DPAK2
- moved R12 24.0 mm to (220.3, 118.0), turned to 270 degrees
- moved R2 20.3 mm to (225.0, 111.9), turned to 90 degrees
- moved D4 19.2 mm to (242.5, 111.4)
- moved TP15 17.0 mm to (205.8, 125.6)
- moved R17 16.4 mm to (238.2, 125.7), turned to 270 degrees
- moved R11 16.3 mm to (223.8, 118.1)
- moved D3 15.2 mm to (221.9, 127.6), turned to 90 degrees
- moved R14 14.1 mm to (234.8, 115.6), turned to 90 degrees
- moved R15 14.0 mm to (244.1, 121.6), turned to 270 degrees
- moved D1 14.0 mm to (237.2, 135.3)
- moved TP17 14.0 mm to (224.2, 121.4)
- moved C10 12.2 mm to (247.3, 114.2), turned to 270 degrees
- moved TP16 11.6 mm to (226.1, 117.1)
- moved Q1 11.5 mm to (226.3, 137.8), turned to 90 degrees
- moved TP5 11.3 mm to (237.2, 106.1)
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Connections:
- net /DigitalAccess/EC_GND renamed /DigitalAccess/VGND
- net /EC/EC_V renamed /DigitalAccess/EC_Meas
- net AC_Signal renamed AC_Shrunk
- D4 pad 1: N-0000057 (its old number) -> N-0000055
- D5 pad 2: N-0000057 (its old number) -> N-0000055
- R13 pad 2: N-0000054 -> N-0000055
- R14 pad 1: N-0000057 (its old number) -> N-0000055
- R15 pad 1: N-0000057 (its old number) -> N-0000055
- TP20 pad 1: N-0000054 -> N-0000055
- U1 pad 7: N-0000054 -> N-0000055
Routing:
- net /DigitalAccess/V+_WallWart: track 15.5 -> 96.4 mm
- net /DigitalAccess/~RESET: track 0.00 -> 71.6 mm, vias 0 -> 1
- net /DigitalAccess/~DR: track 0.00 -> 40.4 mm
- net N-0000041: track 0.00 -> 34.2 mm
- net /DigitalAccess/~CS_ISO: track 0.00 -> 31.9 mm, vias 0 -> 1
- net /DigitalAccess/MISO_ISO: track 0.00 -> 29.9 mm, vias 0 -> 1
- net /DigitalAccess/MOSI_ISO: track 0.00 -> 29.5 mm, vias 0 -> 1
- net /DigitalAccess/EC_Meas: track 0.00 -> 29.1 mm
- net N-0000055: track 0.00 -> 28.1 mm
- net /DigitalAccess/SCLK_ISO: track 0.00 -> 26.6 mm
- net /EC/EC_Probe+: track 28.3 -> 54.4 mm
- net N-0000048: track 0.00 -> 16.9 mm
- net N-0000049: track 0.00 -> 15.8 mm, vias 0 -> 2
- net /Pumps/SW_ECPump: track 20.8 -> 36.5 mm
- net N-0000040: track 5.78 -> 21.4 mm
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- added copper zone on B.Cu, net AGND

Commit message: moved some of the component text from under a component in the layout
Parts:
- D1: value 4004 -> (none)
- D3: value DIODE -> (none)
- P2: value WallWartExtension -> (none)
- X1: value CRYSTAL -> (none)
