File: Kicad/_autosave-HealthyEC.kicad_pcb (KiCad board)
At the start: 2 copper layers, 68.6 x 53.3 mm, 54 parts, among them P1 CONN_4, P2 WallWartExtension, Q1 TIP122, U1 MCP6244, U2 MCP3901, X1 CRYSTAL

Commit message: Started changes for Dev-Rev3
Parts:
- removed RV2, RV3: POT, LB_POT
Routing:
- net AC_Shrunk: track 23.0 -> 12.1 mm
- net EC_Signal: track 21.7 -> 15.0 mm
- net /EC/EC_Probe+: track 41.9 -> 35.9 mm
Changed lines of the file:
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@@
 (kicad_pcb (version 3) (host pcbnew "(2013-07-07 BZR 4022)-stable")
   (general
-    (links 101)
-    (no_connects 0)
+    (links 97)
+    (no_connects 19)
     (area 178.156799 99.655559 253.744801 153.82856)
     (thickness 1.6)
     (drawings 10)
-    (tracks 345)
+    (tracks 330)
     (zones 0)
-    (modules 54)
+    (modules 52)
     (nets 37)
   )
@@
     (visible_elements 7FFFFFFF)
     (pcbplotparams
-      (layerselection 284196865)
+      (layerselection 3178497)
       (usegerberextensions true)
       (excludeedgelayer true)
@@
       (psa4output false)
       (plotreference true)
-      (plotvalue false)
+      (plotvalue true)
       (plotothertext true)
       (plotinvisibletext false)
@@
     )
   )
-  (module LB_POT (layer F.Cu)
-    (at 235.67644 114.80038 180)
-    (fp_text reference RV2 (at 4.7 -0.6 180) (layer F.SilkS)
-      (effects (font (size 1 1) (thickness 0.15)))
-    )
-    (fp_text value POT (at 1.4605 -0.59944 180) (layer F.SilkS)
-      (effects (font (size 1 1) (thickness 0.15)))
-    )
-    (fp_line (start 0 0) (end 0 5.56) (layer F.SilkS) (width 0.15))
-    (fp_line (start 0 5.56) (end 9.78 5.56) (layer F.SilkS) (width 0.15))
-    (fp_line (start 9.78 5.56) (end 9.78 0) (layer F.SilkS) (width 0.15))
-    (fp_line (start 9.78 0) (end 0 0) (layer F.SilkS) (width 0.15))
-    (pad 1 thru_hole circle (at 2.6 2.75 180) (size 1.016 1.016) (drill 0.635)
-      (layers *.Cu *.Mask F.SilkS)
-      (net 32 AC_Shrunk)
-    )
-    (pad 2 thru_hole circle (at 5.2 2.75 180) (size 1.016 1.016) (drill 0.635)
-      (layers *.Cu *.Mask F.SilkS)
-      (net 18 /DigitalAccess/VGND)
-    )
-    (pad 3 thru_hole circle (at 7.8 2.75 180) (size 1.016 1.016) (drill 0.635)
-      (layers *.Cu *.Mask F.SilkS)
-    )
-  )
-  (module LB_POT (layer F.Cu)
-    (at 225.31324 114.75212 180)
-    (fp_text reference RV3 (at 4.7 -0.6 180) (layer F.SilkS)
-      (effects (font (size 1 1) (thickness 0.15)))
-    )
-    (fp_text value POT (at 1.4605 -0.59944 180) (layer F.SilkS)
-      (effects (font (size 1 1) (thickness 0.15)))
-    )
-    (fp_line (start 0 0) (end 0 5.56) (layer F.SilkS) (width 0.15))
-    (fp_line (start 0 5.56) (end 9.78 5.56) (layer F.SilkS) (width 0.15))
-    (fp_line (start 9.78 5.56) (end 9.78 0) (layer F.SilkS) (width 0.15))
-    (fp_line (start 9.78 0) (end 0 0) (layer F.SilkS) (width 0.15))
-    (pad 1 thru_hole circle (at 2.6 2.75 180) (size 1.016 1.016) (drill 0.635)
-      (layers *.Cu *.Mask F.SilkS)
-    )
-    (pad 2 thru_hole circle (at 5.2 2.75 180) (size 1.016 1.016) (drill 0.635)
-      (layers *.Cu *.Mask F.SilkS)
-      (net 34 EC_Signal)
-    )
-    (pad 3 thru_hole circle (at 7.8 2.75 180) (size 1.016 1.016) (drill 0.635)
-      (layers *.Cu *.Mask F.SilkS)
-      (net 22 /EC/EC_Probe+)
-    )
-  )
   (gr_text "Healthy EC\nDev-Rev2" (at 199.65416 103.1367) (layer F.SilkS)
     (effects (font (size 1.5 1.5) (thickness 0.3)))
@@
   (segment (start 222.0087 116.7638) (end 220.1612 116.7638) (width 0.254) (layer F.Cu) (net 22))
   (segment (start 220.1612 116.7638) (end 220.05 116.875) (width 0.254) (layer F.Cu) (net 22))
-  (segment (start 217.32782 111.92338) (end 217.32782 112.73062) (width 0.254) (layer F.Cu) (net 22))
-  (segment (start 220.05 115.4528) (end 220.05 116.875) (width 0.254) (layer F.Cu) (net 22))
-  (segment (start 217.32782 112.73062) (end 220.05 115.4528) (width 0.254) (layer F.Cu) (net 22))
   (segment (start 220.9 120.9) (end 221.95 120.9) (width 0.254) (layer F.Cu) (net 22))
   (segment (start 220.9 120.9) (end 220.05 120.05) (width 0.254) (layer F.Cu) (net 22))
@@
   (segment (start 234.6975 120.5525) (end 235.55 120.5525) (width 0.254) (layer F.Cu) (net 28))
   (segment (start 233.9 121.35) (end 234.6975 120.5525) (width 0.254) (layer F.Cu) (net 28))
-  (segment (start 232.8418 119.5705) (end 234.627 119.5705) (width 0.254) (layer F.Cu) (net 29))
   (segment (start 234.627 119.5705) (end 235.55 118.6475) (width 0.254) (layer F.Cu) (net 29))
+  (segment (start 232.8418 119.5705) (end 234.627 119.5705) (width 0.254) (layer F.Cu) (net 29))
   (segment (start 230.10114 118.27256) (end 230.57104 118.27256) (width 0.254) (layer F.Cu) (net 29))
   (segment (start 231.86898 119.5705) (end 232.8418 119.5705) (width 0.254) (layer F.Cu) (net 29))
@@
   (segment (start 246.25808 142.42034) (end 243.21262 142.42034) (width 0.6096) (layer F.Cu) (net 31))
   (segment (start 249.018 139.66042) (end 246.25808 142.42034) (width 0.6096) (layer F.Cu) (net 31))
-  (segment (start 232.70718 112.3188) (end 232.84104 112.3188) (width 0.254) (layer F.Cu) (net 32))
-  (segment (start 232.84104 112.3188) (end 233.15518 112.00466) (width 0.254) (layer F.Cu) (net 32))
-  (segment (start 230.6066 114.4016) (end 230.62438 114.4016) (width 0.254) (layer F.Cu) (net 32))
-  (segment (start 229.71633 115.29187) (end 230.6066 114.4016) (width 0.254) (layer F.Cu) (net 32))
-  (segment (start 230.62438 114.4016) (end 232.70718 112.3188) (width 0.254) (layer F.Cu) (net 32))
-  (segment (start 232.70718 112.3188) (end 232.76052 112.26546) (width 0.254) (layer F.Cu) (net 32))
   (segment (start 231.91216 116.97462) (end 231.39908 116.97462) (width 0.254) (layer F.Cu) (net 32))
-  (segment (start 231.39908 116.97462) (end 229.71633 115.29187) (width 0.254) (layer F.Cu) (net 32))
   (segment (start 231.79786 117.29466) (end 231.71912 117.29466) (width 0.254) (layer F.Cu) (net 32))
-  (segment (start 228.19614 118.27256) (end 228.19614 116.81206) (width 0.254) (layer F.Cu) (net 32))
-  (segment (start 228.19614 116.81206) (end 229.71633 115.29187) (width 0.254) (layer F.Cu) (net 32))
   (segment (start 226.31908 124.2568) (end 227.9182 124.2568) (width 0.254) (layer F.Cu) (net 32))
   (segment (start 228.19614 120.29614) (end 228.19614 118.27256) (width 0.254) (layer F.Cu) (net 32))
@@
   (segment (start 223.9137 116.7638) (end 223.9137 118.61038) (width 0.254) (layer F.Cu) (net 34))
   (segment (start 223.9137 118.61038) (end 222.86214 119.66194) (width 0.254) (layer F.Cu) (net 34))
-  (segment (start 219.92782 111.92338) (end 220.2112 111.92338) (width 0.254) (layer F.Cu) (net 34))
-  (segment (start 223.9137 115.62588) (end 223.9137 116.7638) (width 0.254) (layer F.Cu) (net 34))
-  (segment (start 220.2112 111.92338) (end 223.9137 115.62588) (width 0.254) (layer F.Cu) (net 34))
   (segment (start 226.31908 121.7168) (end 224.2668 121.7168) (width 0.254) (layer F.Cu) (net 34))
   (segment (start 224.2668 121.7168) (end 224.125 121.575) (width 0.254) (layer F.Cu) (net 34))
